Commit message: Add exca_autodig

File: exca_bringup/urdf/exca_urdf.urdf.xacro (robot description, xacro)
@@ -6,5 +6,5 @@
     <axis xyz="0 0 1"/>
     <limit effort="1000.0" lower="0.0" upper="6.28318" velocity="0.5"/>
-    <origin rpy="0 0 0" xyz="0.0 0.0 0.155"/>
+    <origin rpy="0 0 -1.5708" xyz="0.0 0.0 0.163"/>
     <parent link="base_footprint"/>
     <child link="swing_frame"/>
@@ -14,5 +14,5 @@
     <axis xyz="0 0 1"/>
     <limit effort="1000.0" lower="0.0" upper="6.28318" velocity="0.5"/>
-    <origin rpy="1.5708 0 -1.5708" xyz="0.05 0.0 0.0"/>
+    <origin rpy="1.5708 0 -1.5708" xyz="0.0 0.0 0.0"/>
     <parent link="swing_frame"/>
     <child link="boom_frame"/>
@@ -22,5 +22,5 @@
     <axis xyz="0 0 1"/>
     <limit effort="1000.0" lower="0.0" upper="6.28318" velocity="0.5"/>
-    <origin rpy="0 0 0" xyz="-0.21 0.39 0.0"/>
+    <origin rpy="0 0 0" xyz="-0.205 0.424 0.0"/>
     <parent link="boom_frame"/>
     <child link="arm_frame"/>
@@ -30,5 +30,5 @@
     <axis xyz="0 0 1"/>
     <limit effort="1000.0" lower="0.0" upper="6.28318" velocity="0.5"/>
-    <origin rpy="0 0 0" xyz="-0.19 0.185 0.0"/>
+    <origin rpy="0 0 0" xyz="-0.192 0.14 0.0"/>
     <parent link="arm_frame"/>
     <child link="bucket_frame"/>
@@ -36,5 +36,5 @@
   <link name="bucket_frame"/>
   <joint name="tip_joint" type="fixed">
-      <origin rpy="0 0.0 0.0" xyz="-0.05 0.15 0"/>
+      <origin rpy="0 0.0 0.0" xyz="-0.055 0.153 0"/>
       <parent link="bucket_frame"/>
       <child link="bucket_tip"/>
