Commit message: Add urdf and others

File: elavation_mapping_test/urdf/scanner.urdf.xacro (robot description, xacro)
@@ -6,5 +6,5 @@
       <axis xyz="0 1 0"/>
       <limit effort="1000.0" lower="0.0" upper="3.14159" velocity="0.5"/>
-      <origin rpy="0 0 0" xyz="0.0 0.0 0.9"/>
+      <origin rpy="0 0 0" xyz="0.0 0.0 0.4"/>
       <parent link="laser_base"/>
       <child link="scanner_link"/>
@@ -12,5 +12,5 @@
   <link name="scanner_link"/>
   <joint name="laser_joint" type="fixed">
-      <origin rpy="3.141593 0.0 3.141593" xyz="0.0 0.0 -0.003"/>
+      <origin rpy="3.141593 1.6008 3.141593" xyz="0.0 0.0 0.0"/>
       <parent link="scanner_link"/>
       <child link="laser_frame"/>

Commit message: New Progress

File: elavation_mapping_test/urdf/scanner.urdf.xacro (robot description, xacro)
@@ -6,5 +6,5 @@
       <axis xyz="0 1 0"/>
       <limit effort="1000.0" lower="0.0" upper="3.14159" velocity="0.5"/>
-      <origin rpy="0 0 0" xyz="0.0 0.0 0.4"/>
+      <origin rpy="0 0 0" xyz="0.0 0.0 0.485"/>
       <parent link="laser_base"/>
       <child link="scanner_link"/>

File: exca_bringup/urdf/exca_urdf.urdf.xacro (robot description, xacro)
@@ -6,5 +6,5 @@
     <axis xyz="0 0 1"/>
     <limit effort="1000.0" lower="0.0" upper="6.28318" velocity="0.5"/>
-    <origin rpy="0 0 -1.5708" xyz="0.0 0.0 0.163"/>
+    <origin rpy="0.0 0 -1.5708" xyz="0.0 0.0 0.163"/>
     <parent link="base_footprint"/>
     <child link="swing_frame"/>
